File: hardware/red-scout-aa.sch (KiCad schematic (older format))
At the start: 36 parts, among them P1 SNAP, P10 CONN_01X06, P2 SNAP, P3 SNAP, P4 SNAP, P5 SNAP, P6 SNAP, P7 SNAP, P8 SNAP, P9 IO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

Commit message: Label UART1 header.
Parts:
- P10: value CONN_01X06 -> UART1
Changed lines of the file:
@@
 P 7050 3100
 F 0 "P10" H 7050 3450 50  0000 C CNN
-F 1 "CONN_01X06" V 7150 3100 50  0000 C CNN
+F 1 "UART1" V 7150 3100 50  0000 C CNN
 F 2 "" H 7050 3100 60  0000 C CNN
 F 3 "" H 7050 3100 60  0000 C CNN
